File: PCB/AnalogIsolator/AnalogIsolator/AnalogIsolator.kicad_pcb (KiCad board)
At the start: 0 parts

Commit message: update: fix design pcb
Parts:
- added C1: 100nf, Capacitor_SMD:C_0603_1608Metric, F.Cu at (121.5, 52.6)
- added C10: 100nf, Capacitor_SMD:C_0603_1608Metric, F.Cu at (98.8, 65.7)
- added C2: 2.2nf COG, Capacitor_SMD:C_0603_1608Metric, F.Cu at (104.0, 65.7)
- added C3: 100nf, Capacitor_SMD:C_0603_1608Metric, F.Cu at (101.8, 48.2)
- added C4: 4.7uf, Capacitor_SMD:C_0603_1608Metric, F.Cu at (101.8, 49.8)
- added C5: 10uf, Capacitor_SMD:C_0805_2012Metric, F.Cu at (116.3, 52.6)
- added C6: 100nf, Capacitor_SMD:C_0603_1608Metric, F.Cu at (125.2, 55.4)
- added C7: 1nf COG, Capacitor_SMD:C_0603_1608Metric, F.Cu at (126.5, 64.4)
- added C8: 100nf, Capacitor_SMD:C_0603_1608Metric, F.Cu at (98.2, 58.5)
- added C9: 100nf, Capacitor_SMD:C_0603_1608Metric, F.Cu at (123.7, 60.6)
- added D2: LED, LED_SMD:LED_0603_1608Metric, F.Cu at (97.8, 46.6)
- added L1: BLM18AG601SN1D, footprint:L0603, F.Cu at (101.8, 51.4)
- added M2.4V1: 0, Resistor_SMD:R_0603_1608Metric, F.Cu at (100.7, 61.7)
- added M3.3V1: 0, Resistor_SMD:R_0603_1608Metric, F.Cu at (102.4, 61.7)
- added M5V1: 0, Resistor_SMD:R_0603_1608Metric, F.Cu at (104.0, 61.7)
- added R1: 4.7k, Resistor_SMD:R_0603_1608Metric, F.Cu at (125.2, 57.0)
- added R10: 100k 1%, Resistor_SMD:R_0603_1608Metric, F.Cu at (94.1, 49.3)
- added R11: 1k 0.1%, Resistor_SMD:R_0603_1608Metric, F.Cu at (98.6, 61.7)
- added R2: 164k 0.1%, Resistor_SMD:R_0603_1608Metric, F.Cu at (122.0, 57.0)
- added R3: 220, Resistor_SMD:R_0603_1608Metric, F.Cu at (120.9, 64.4)
- added R4: 80.6k 0.1%, Resistor_SMD:R_0805_2012Metric, F.Cu at (100.0, 58.4)
- added R5: 101k 0.1%, Resistor_SMD:R_0805_2012Metric, F.Cu at (102.0, 58.4)
- added R6: 150k 0.1%, Resistor_SMD:R_0805_2012Metric, F.Cu at (104.0, 58.4)
- added R7: 1k, Resistor_SMD:R_0603_1608Metric, F.Cu at (101.8, 46.6)
- added R9: 1.8k 0.1%, Resistor_SMD:R_0805_2012Metric, F.Cu at (104.0, 53.7)
- added U1: HCNR201-500E, footprint:OPTO-SMD-8P_L11.0-W9.0-P2.54-LS12.4-BL, F.Cu at (112.4, 59.8)
- added U3: OPA317IDBVR-TP, footprint:SOT-23-5_L2.9-W1.6-P0.95-LS2.8-BR, F.Cu at (101.5, 65.7)
- added U4: IF0505S-1WR3_C5369637, footprint:PWRM-TH_BXXXXLS-1W, F.Cu at (113.8, 46.4)
- added U5: OPA392DBVR, footprint:SOT-23-5_L2.9-W1.6-P0.95-LS2.8-BL, F.Cu at (123.7, 64.4)
- added U7: AO3401A_C347476, footprint:SOT-23_L2.9-W1.3-P1.90-LS2.4-BR, F.Cu at (97.7, 49.7)
- added U8: KF301-5_0-3P, footprint:CONN-TH_3P-P5.00_KF301-5.0-3P, F.Cu at (92.4, 59.6)
- added U9: KF301-5_0-3P, footprint:CONN-TH_3P-P5.00_KF301-5.0-3P, F.Cu at (132.3, 60.0)
Routing:
- net +5V_ISO: track 0.00 -> 66.5 mm
- net +5V_HOST: track 0.00 -> 41.6 mm
- net /SUM2: track 0.00 -> 33.0 mm
- net +5V: track 0.00 -> 26.0 mm, vias 0 -> 1
- net Net-(U3-OUT): track 0.00 -> 19.6 mm
- net /SUM1: track 0.00 -> 16.5 mm
- net /AOUT: track 0.00 -> 11.9 mm
- net Net-(U5-OUT): track 0.00 -> 10.0 mm
- net Net-(U4-VIN): track 0.00 -> 9.75 mm
- net /AIN: track 0.00 -> 7.82 mm
- net GND: track 0.00 -> 6.39 mm, vias 0 -> 8
- net Net-(C6-Pad1): track 0.00 -> 3.17 mm
- net Net-(U7-G): track 0.00 -> 3.00 mm
- net Net-(R6-Pad2): track 0.00 -> 2.80 mm
- net Net-(U1-L_CAT): track 0.00 -> 2.53 mm
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- added copper zone on B.Cu, net GND
- added copper zone on F.Cu, net GND
- added copper zone on B.Cu, net GND_ISO
- added copper zone on F.Cu, net GND_ISO
Other:
- board outline added: 48 x 32.4 mm
- copper layers 0 -> 2
- board text added: "5V 200mA ISOLATED"
- board text added: "AIN GND 5V"
- board text added: "AOUT GND 5V"
- board text added: "FIT ONE ONLY"
- board text added: "MCU SIDE"
- board text added: "SENSOR SIDE"
