File: PCB/AnalogIsolator/AnalogIsolator/AnalogIsolator.kicad_sch (KiCad schematic)
At the start: 28 parts, among them J1 Conn_01x03_Pin, J2 Conn_01x03_Pin, U1 HCNR201-500E, U2 OPA317M/TR, U3 OPA317M/TR, U4 IF0505S-1WR3_C5369637, U5 BAV199,215, U6 BAV199,215, U7 AO3401A_C347476, U8 KF301-5_0-3P, U9 KF301-5_0-3P

Commit message: update: fix schematic
Parts:
- removed D1: 1N4148WS-C57759, footprint:SOD-323_L1.8-W1.3-LS2.5-RD-1, symbol lcsc:1N4148WS-C57759
- removed J1, J2: Conn_01x03_Pin, symbol Connector:Conn_01x03_Pin
- removed R8: 249 0.25W, symbol Device:R
- removed U2, U3: OPA317M/TR, footprint:SOIC-8_L4.9-W3.9-P1.27-LS6.0-BL, symbol lcsc:OPA317M/TR
- removed U5, U6: BAV199,215, footprint:SOT-23-3_L3.0-W1.7-P0.95-LS2.9-BR, symbol lcsc:BAV199,215
- added C10, C6, C8, C9: 100nf, symbol Device:C
- added C7: 1nf COG, symbol Device:C
- added D2: LED, symbol Device:LED
- added R11: 1k 0.1%, symbol Device:R
- added SW1: SW_SP3T, symbol Switch:SW_SP3T
- added U3: OPA317IDBVR-TP, footprint:SOT-23-5_L2.9-W1.6-P0.95-LS2.8-BR, symbol lcsc:OPA317IDBVR-TP
- added U5: OPA392DBVR, footprint:SOT-23-5_L2.9-W1.6-P0.95-LS2.8-BL, symbol lcsc:OPA392DBVR
- C1: value 1nf COG -> 100nf
- C3: value 100nf X7R -> 100nf
- C4: value 4.7uf X5R -> 4.7uf
- C5: value 10uf X5R -> 10uf
Connections:
- net at R9.1: now also R6.2
- net SUM2: now reaches R9.2
- net SUM2: now also C2.1, R4.2, R5.2, U1.6 (PD2_CAT), U3.4 (-IN)
- net at R7.1: now also D2.2 (A)
- net at R7.2: now also C3.1, C4.1, L1.2, U4.1 (VIN)
- net at U1.1 (L_CAT): now also R3.2
- net +5V_ISO: now reaches U1.2 (L_AN)
- net +5V_ISO: now also C1.1, C5.1, U4.6 (+VO), U9.1, C9.1, U5.5 (V+)
- net SUM1: now reaches U1.3 (PD1_CAT)
- net SUM1: now also R2.2, C7.1, U5.4 (IN_-)
- net GND_ISO: now reaches U1.4 (PD1_AN)
- net GND_ISO: now also C1.2, C5.2, U4.4 (-VO), U9.2, C6.2, C9.2, U5.2 (V-), U5.3 (IN_+)
- net GND: now reaches U1.5 (PD2_AN)
- net GND: now also C3.2, C4.2, R10.2, U4.2 (GND), U8.2, C10.2, C8.2, D2.1 (K), U3.2 (V-), U3.3 (+IN)
- net +5V_HOST: now reaches L1.1
- net +5V_HOST: now also U7.2 (S), C10.1, U3.5 (V+)
- net at R4.1: now also SW1.4
- net at R10.1: now also U7.1 (G)
- net at R2.1: now also R1.2, C6.1
- net AOUT: now reaches U8.1
- net AOUT: now also C8.1, R11.2
- net +5V: now reaches U8.3
- net +5V: now also U7.3 (D)
- net AIN: now reaches U9.3
- net AIN: now also R1.1
- net at R6.1: now also SW1.1
- net at C2.2: now also R11.1, SW1.3, U3.1 (OUT)
- net at R3.1: now also C7.2, U5.1 (OUT)
- net at R5.1: now also SW1.2
- no-connect marks 0 -> 2
Other:
- moved on the sheet: C1, C2, C3, C4, C5, L1, R1, R10, R2, R3, R4, R5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

Commit message: update: fix design pcb
Parts:
- removed SW1: SW_SP3T, symbol Switch:SW_SP3T
- added M2.4V1, M3.3V1, M5V1: 0, Resistor_SMD:R_0603_1608Metric, symbol Device:R
- C1, C10, C2, C3, C4, C6, C7, C8, C9: footprint (none) -> Capacitor_SMD:C_0603_1608Metric
- C5: footprint (none) -> Capacitor_SMD:C_0805_2012Metric
- R1, R10, R11, R2, R3, R7: footprint (none) -> Resistor_SMD:R_0603_1608Metric
- R4, R5, R6, R9: footprint (none) -> Resistor_SMD:R_0805_2012Metric
Connections:
- net at R6.1: now also M5V1.2
- net at R5.1: now also M3.3V1.2
- net at C2.2, R11.1, U3.1 (OUT): now also M2.4V1.1, M3.3V1.1, M5V1.1
- net at R4.1: now also M2.4V1.2
